Commit message: psd等の修正完了、トピック名も変更

File: tum_simulator/cvg_sim_gazebo/urdf/quadrotor_psd.urdf.xacro (robot description, xacro)
@@ -17,16 +17,16 @@
 	<!-- psd sensor -->
 	<xacro:include filename="$(find cvg_sim_gazebo)/urdf/sensors/psd_sensor.urdf.xacro" />
-	<xacro:psd_sensor name="psd_left" parent="base_link" ros_topic="psd_left" update_rate="30" min_range="0.01" max_range="0.5" ray_count="2" visualize="true">
+	<xacro:psd_sensor name="psd_left" parent="base_link" ros_topic="front_left" update_rate="30" sim_name="ardrone" min_range="0.01" max_range="0.5" ray_count="2" visualize="true">
       <origin xyz="0.26 0.14 0.02" rpy="0 0 0"/>
     </xacro:psd_sensor>
-	<xacro:psd_sensor name="psd_right" parent="base_link" ros_topic="psd_right" update_rate="30" min_range="0.01" max_range="0.5" ray_count="2" visualize="true">
+	<xacro:psd_sensor name="psd_right" parent="base_link" ros_topic="front_right" update_rate="30" sim_name="ardrone" min_range="0.01" max_range="0.5" ray_count="2" visualize="true">
       <origin xyz="0.26 -0.14 0.02" rpy="0 0 0"/>
 	  <!-- <origin xyz="0.26 -0.14 0.02" rpy="0 ${90*M_PI/180} 0"/> -->
     </xacro:psd_sensor>
-	<xacro:psd_sensor name="psd_left_side" parent="base_link" ros_topic="psd_left_side" update_rate="30" min_range="0.01" max_range="0.5" ray_count="2" visualize="true">
+	<xacro:psd_sensor name="psd_left_side" parent="base_link" ros_topic="left_side" update_rate="30" sim_name="ardrone" min_range="0.01" max_range="0.5" ray_count="2" visualize="true">
       <origin xyz="0.0 0.24 0.02" rpy="0 0 ${90*M_PI/180}"/>
 	  <!-- <origin xyz="0.26 -0.14 0.02" rpy="0 ${90*M_PI/180} 0"/> -->
     </xacro:psd_sensor>
-	<xacro:psd_sensor name="psd_right_side" parent="base_link" ros_topic="psd_right_side" update_rate="30" min_range="0.01" max_range="0.5" ray_count="2" visualize="true">
+	<xacro:psd_sensor name="psd_right_side" parent="base_link" ros_topic="right_side" update_rate="30" sim_name="ardrone" min_range="0.01" max_range="0.5" ray_count="2" visualize="true">
       <origin xyz="0. -0.24 0.02" rpy="0 0 -${90*M_PI/180}"/>
 	  <!-- <origin xyz="0.26 -0.14 0.02" rpy="0 ${90*M_PI/180} 0"/> -->

File: tum_simulator/cvg_sim_gazebo/urdf/sensors/psd_sensor.urdf.xacro (robot description, xacro)
@@ -8,5 +8,5 @@
   <property name="M_PI" value="3.1415926535897931" />
   <property name="field_of_view" value="${1*M_PI/180}" />
-  <xacro:macro name="psd_sensor" params="name parent *origin ros_topic update_rate min_range max_range ray_count visualize">
+  <xacro:macro name="psd_sensor" params="name parent *origin ros_topic update_rate sim_name min_range max_range ray_count visualize">
 	<joint name="${name}_joint" type="fixed">
       <xacro:insert_block name="origin" />
@@ -68,5 +68,5 @@
         <plugin name="gazebo_ros_${name}_controller" filename="libhector_gazebo_ros_sonar.so">
           <gaussianNoise>0.000</gaussianNoise>
-          <topicName>${ros_topic}</topicName>
+          <topicName>${sim_name}/psd/${ros_topic}</topicName>
           <frameId>${name}_link</frameId>
         </plugin>
