Commit message: base_linkをardrone_base_linkに変更中

File: tum_simulator/cvg_sim_gazebo/urdf/quadrotor.urdf (robot description, URDF)
Before this commit: robot quadrotor, 1 links, 0 joints
Links:
- removed link base_link
- added link ardrone_base_link, mass 1.477; collision mesh filename=package://cvg_sim_gazebo/meshes/quadrotor/quadrotor_4.stl; visual mesh filename=package://cvg_sim_gazebo/meshes/quadrotor/quadrotor_4.dae

File: tum_simulator/cvg_sim_gazebo/urdf/quadrotor_base.urdf.xacro (robot description, xacro)
@@ -9,5 +9,5 @@
   <!-- Main quadrotor link -->
   <xacro:macro name="quadrotor_base_macro">
-    <link name="base_link">
+    <link name="ardrone_base_link">
       <inertial>
         <mass value="1.477" />
@@ -28,5 +28,5 @@
       </collision>
     </link>
-    <gazebo reference="base_link">
+    <gazebo reference="ardrone_base_link">
       <turnGravityOff>false</turnGravityOff>
     </gazebo>

File: tum_simulator/cvg_sim_gazebo/urdf/quadrotor_sensors.urdf (robot description, URDF)
Before this commit: robot quadrotor_hokuyo_utm30lx, 2 links, 1 joints
Links:
- removed link base_link
- added link ardrone_base_link; visual mesh filename=package://cvg_sim_gazebo/meshes/quadrotor/quadrotor_4.dae
Joints:
- joint sonar_joint: parent base_link -> ardrone_base_link

File: tum_simulator/cvg_sim_gazebo_plugins/urdf/quadrotor_plugins.urdf.xacro (robot description, xacro)
@@ -5,5 +5,5 @@
   <!-- Quadrotor Gazebo Plugins -->
   <xacro:macro name="quadrotor_plugins">
-    <canonicalBody>base_link</canonicalBody>
+    <canonicalBody>ardrone_base_link</canonicalBody>
     <quadrotor_sensors/>
     <quadrotor_controller/>

File: tum_simulator/cvg_sim_gazebo_plugins/urdf/quadrotor_sensors.urdf.xacro (robot description, xacro)
@@ -13,5 +13,5 @@
         <alwaysOn>true</alwaysOn>
         <updateRate>100.0</updateRate>
-        <bodyName>base_link</bodyName>
+        <bodyName>ardrone_base_link</bodyName>
         <frameId>ardrone_base_link</frameId>
         <topicName>/ardrone/imu</topicName>
@@ -28,5 +28,5 @@
         <alwaysOn>true</alwaysOn>
         <updateRate>10.0</updateRate>
-        <bodyName>base_link</bodyName>
+        <bodyName>ardrone_base_link</bodyName>
         <topicName>pressure_height</topicName>
         <altimeterTopicName>altimeter</altimeterTopicName>
@@ -38,5 +38,5 @@
         <alwaysOn>true</alwaysOn>
         <updateRate>10.0</updateRate>
-        <bodyName>base_link</bodyName>
+        <bodyName>ardrone_base_link</bodyName>
         <topicName>magnetic</topicName>
         <offset>0 0 0</offset>
@@ -47,5 +47,5 @@
         <alwaysOn>true</alwaysOn>
         <updateRate>4.0</updateRate>
-        <bodyName>base_link</bodyName>
+        <bodyName>ardrone_base_link</bodyName>
         <topicName>fix</topicName>
         <velocityTopicName>fix_velocity</velocityTopicName>
@@ -58,5 +58,5 @@
         <alwaysOn>true</alwaysOn>
         <updateRate>100.0</updateRate>
-        <bodyName>base_link</bodyName>
+        <bodyName>ardrone_base_link</bodyName>
         <topicName>ground_truth/state</topicName>
         <gaussianNoise>0.0</gaussianNoise>

File: tum_simulator/cvg_sim_gazebo_plugins/urdf/quadrotor_simple_controller.urdf.xacro (robot description, xacro)
@@ -10,5 +10,5 @@
         <alwaysOn>true</alwaysOn>
         <updateRate>0.0</updateRate>
-        <bodyName>base_link</bodyName>
+        <bodyName>ardrone_base_link</bodyName>
         <stateTopic>ground_truth/state</stateTopic>
         <imuTopic>ardrone/imu</imuTopic>
@@ -34,5 +34,5 @@
         <alwaysOn>true</alwaysOn>
         <updateRate>0.0</updateRate>
-        <bodyName>base_link</bodyName>
+        <bodyName>ardrone_base_link</bodyName>
         <stateTopic>ground_truth/state</stateTopic>
         <imuTopic>ardrone/imu</imuTopic>
